File: eda/rack-manager/rack-manager/rack-manager.kicad_sch (KiCad schematic)
At the start: 96 parts, among them J1 Screw_Terminal_01x02, J10 Screw_Terminal_01x02, J11 Conn_02x03_Odd_Even, J12 Conn_01x02_Pin, J13 Conn_01x04_Socket, J16 Conn_01x04_Socket, J17 Conn_01x04_Socket, J18 Conn_01x04_Socket, J19 Conn_01x04_Socket, J2 Screw_Terminal_01x02, J20 Conn_01x04_Socket, J21 Conn_01x04_Socket, J22 Conn_01x04_Socket, J23 Conn_01x04_Socket, J24 Conn_02x06_Odd_Even, J25 Conn_02x06_Odd_Even, J3 Screw_Terminal_01x02, J4 Screw_Terminal_01x02, J5 Screw_Terminal_01x02, J6 Screw_Terminal_01x02, J7 Screw_Terminal_01x02, J8 Screw_Terminal_01x02, J9 Screw_Terminal_01x02, SW1 C720477, U5 TCA9548AMRGER, U6 PCA9555PW

Commit message: Final PCB design, work on 3D cad files
Parts:
- added C22: 200uF, Capacitor_THT:CP_Radial_D8.0mm_P3.50mm, symbol Device:C_Small
- ADC1, ADC2, ADC3: LCSC (none) -> C5215160
- H1, H2, H3: now not fitted
- SW1: LCSC (none) -> C720477
Connections:
- net +5V: now also C22.1
- net GND: now also C22.2
Other:
- moved on the sheet: J10
